File: kicad/sinte555/sinte555.kicad_sch (KiCad schematic)
At the start: 10 parts, among them U1 NE555P, U2 NE555P

Commit message: agregar nueva version
Parts:
- removed C1: 103_Ceramic, Capacitor_THT:C_Disc_D5.0mm_W2.5mm_P2.50mm, symbol PCM_SL_Capacitors:103_Ceramic
- removed C2: 10uF_16V, Capacitor_THT:CP_Radial_D5.0mm_P2.00mm, symbol PCM_SL_Capacitors:10uF_16V
- removed R2: 500k, symbol Device:R_Variable
- removed R3: 4.7k, symbol Device:R
- removed U1, U2: NE555P, Package_DIP:DIP-8_W7.62mm, symbol Timer:NE555P
- removed V1: 9, symbol Simulation_SPICE:VDC
- added C1: 10n, Capacitor_THT:C_Disc_D5.0mm_W2.5mm_P2.50mm, symbol PCM_SL_Capacitors:100nF_Ceramic
- added C2, C4: 100n, Capacitor_THT:C_Disc_D5.0mm_W2.5mm_P2.50mm, symbol PCM_SL_Capacitors:100nF_Ceramic
- added R2: 10k, symbol Device:R
- added RV1, RV2: 470k, symbol Device:R_Potentiometer
- added U1, U2: NE555D, Package_SO:SOIC-8_3.9x4.9mm_P1.27mm, symbol Timer:NE555D
- C3: value 100nF_Ceramic -> 10n
- R1: value 1k -> 10k
Connections:
- net GND: now also C1.1, C2.1, C4.1, U1.1 (GND), U2.1 (GND)
- net VCC: now also R1.1, RV2.2, U1.4 (~{RST}), U1.8 (VCC), U2.4 (~{RST}), U2.8 (VCC)
- net at LS1.1: now also U2.3 (OUT)
- net at R1.2: now also RV1.2, U1.7 (DISCH); no longer R1.1
- net at C3.2: now also R2.2, U2.6 (THRES), U2.7 (DISCH)
- new net: C1.2, RV1.3, U1.2 (TRIG), U1.6 (THRES)
- new net: U1.3 (OUT), U2.2 (TRIG)
- new net: C2.2, U1.5 (CONT)
- new net: C4.2, U2.5 (CONT)
- new net: R2.1, RV2.3
- no-connect marks 0 -> 2
Other:
- note added: "555 derecha modo monostable 1: a GND 2: a 555 izquierda patita 3 3: a salida por C 100u polarizado 4: a VCC 5: a GND por C 100n 6: a GND por C 100n, a VCC por R de 1k y pote2 470k 7: a 6 8: a VCC"
- note added: "555 izquierda modo astable 1: a GND 2: a GND por C 10n, a pote 1 patita 3 3: a 555 derecha, patita 2 4: a VCC 5: a GND por C de 100n 6: a 2 7: a VCC por R 10k, a pote1 patita 2 8: a VCC"

Commit message: corregir valor
Parts:
- C3: value 10n -> 100n
Changed lines of the file:
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@@
 			)
 		)
-		(property "Value" "10n"
+		(property "Value" "100n"
 			(at 93.98 78.7399 90)
 			(show_name no)
